File: Display ILI.sch (KiCad schematic (older format))
At the start: 0 parts

Commit message: Pheripherial added 22.12.21
Added display connector, I2C connector, button and MAX3485
Parts:
- added C?: 0.1uF, Capacitor_SMD:C_0805_2012Metric, symbol Device:C
- added C?: 10uF, Capacitor_SMD:C_0805_2012Metric, symbol Device:C
- added J?: Conn_01x40_Female, Connector_FFC-FPC:Hirose_FH12-40S-0.5SH_1x40-1MP_P0.50mm_Horizontal, symbol Connector:Conn_01x40_Female
Connections:
- net labels added: +3.3V, CTP_SCL, CTP_SDA, DB0, DB1, DB2, DB3, DB4, DB5, DB6, DB7, GND, SCL, SDA, TFT_CS, TFT_RD, TFT_RS, TFT_RST, TFT_WR
- wire segments 0 -> 74
