File: Display ILI.sch (KiCad schematic (older format))
At the start: 3 parts

Commit message: 24.12.21
Board layout added, Step file added
Parts:
- added R10, R9: 10k, Resistor_SMD:R_0402_1005Metric_Pad0.72x0.64mm_HandSolder, symbol Device:R
- C10, C9: renamed from C?; footprint Capacitor_SMD:C_0805_2012Metric -> Capacitor_SMD:C_0402_1005Metric_Pad0.74x0.62mm_HandSolder
- gave numbers to parts that had none: 1
Connections:
- net labels added: CTP_INT, TFT_AO, TFT_SCLK, TFT_SDI
- net labels removed: DB0, DB1, DB2, DB3, DB4, DB5, DB6, DB7, TFT_RD, TFT_RS, TFT_WR
- wire segments 74 -> 92
Other:
- moved on the sheet: C10, C9
