File: ESP32_BoardV1.sch (KiCad schematic (older format))
At the start: 31 parts, among them J1 Barrel_Jack_Switch, J2 ISP, J3 GPIO expanded, J4 sensor, J5 I2C extended, J7 Display, Q1 UMH3N, SW1 SW_SPDT, U1 AZ1117-3.3, U2 ESP32-WROOM-32E(8MB)

Commit message: PCB completed
Parts:
- removed JP2: SolderJumper_2_Open, Resistor_SMD:R_0402_1005Metric_Pad0.72x0.64mm_HandSolder, symbol Jumper:SolderJumper_2_Open
Connections:
- net labels removed: GPIO32
- wire segments 197 -> 195
Other:
- moved on the sheet: C7, R2, SW1
Changed lines of the file:
@@
 	7400 3750 7550 3750
 Wire Wire Line
-	7400 4150 7550 4150
-Wire Wire Line
 	7400 4450 7550 4450
 Wire Wire Line
@@
 Text Label 6050 2750 2    50   ~ 0
 IO39
-$Comp
-L power:+5V #PWR?
-U 1 1 5F99E8D0
-P 10075 3750
-AR Path="/5E88A377/5F99E8D0" Ref="#PWR?"  Part="1"
-AR Path="/5F99E8D0" Ref="#PWR020"  Part="1"
-AR Path="/5F818C22/5F99E8D0" Ref="#PWR?"  Part="1"
-F 0 "#PWR020" H 10075 3600 50  0001 C CNN
-F 1 "+5V" H 10090 3923 50  0000 C CNN
-F 2 "" H 10075 3750 50  0001 C CNN
-F 3 "" H 10075 3750 50  0001 C CNN
-	1    10075 3750
-	-1   0    0    -1
-$EndComp
 Wire Wire Line
 	10075 3750 10350 3750
@@
 	-1   0    0    -1
 $EndComp
-Text Label 10150 3850 2    50   ~ 0
+Text Label 10150 3950 2    50   ~ 0
 GAS_AOUT
 Wire Wire Line
 	10350 3950 10150 3950
-Text Label 10150 3950 2    50   ~ 0
+Text Label 10150 3850 2    50   ~ 0
 SHARP_AOUT
 Text Label 10150 4050 2    50   ~ 0
@@
 Text Label 8050 4750 0    50   ~ 0
 GAS_AOUT
-Text Label 8050 4350 0    50   ~ 0
-MODBUS_EN
-Text Label 7575 4050 0    50   ~ 0
-MODBUS_TXD
-Text Label 8050 4250 0    50   ~ 0
-MODBUS_RXD
 Text Label 7550 2550 0    50   ~ 0
 UART0_TXD
@@
 	7400 4250 8050 4250
 Wire Wire Line
-	7400 4350 8050 4350
-Wire Wire Line
 	7400 4750 8050 4750
 Wire Wire Line
@@
 $EndComp
 $Comp
-L Jumper:SolderJumper_2_Open JP2
-U 1 1 61C9B3AB
-P 9750 1200
-F 0 "JP2" V 9750 1268 50  0000 L CNN
-F 1 "SolderJumper_2_Open" V 9795 1268 50  0001 L CNN
-F 2 "Resistor_SMD:R_0402_1005Metric_Pad0.72x0.64mm_HandSolder" H 9750 1200 50  0001 C CNN
-F 3 "~" H 9750 1200 50  0001 C CNN
-	1    9750 1200
-	0    1    1    0
-$EndComp
-Connection ~ 9750 1350
-Wire Wire Line
-	9750 1350 10150 1350
-Wire Wire Line
-	9500 1350 9750 1350
-$Comp
 L power:+3.3V #PWR?
 U 1 1 61C9C7C1
@@
 $EndComp
 $Comp
-L power:+5V #PWR?
-U 1 1 61C9DCD6
-P 9750 1050
-AR Path="/5E88A377/61C9DCD6" Ref="#PWR?"  Part="1"
-AR Path="/61C9DCD6" Ref="#PWR018"  Part="1"
-AR Path="/5F818C22/61C9DCD6" Ref="#PWR?"  Part="1"
-F 0 "#PWR018" H 9750 900 50  0001 C CNN
-F 1 "+5V" H 9765 1223 50  0000 C CNN
-F 2 "" H 9750 1050 50  0001 C CNN
-F 3 "" H 9750 1050 50  0001 C CNN
-	1    9750 1050
-	1    0    0    -1
-$EndComp
-$Comp
 L Switch:SW_SPDT SW1
 U 1 1 61CA3FF0
-P 8475 3350
-F 0 "SW1" H 8475 3635 50  0000 C CNN
-F 1 "SW_SPDT" H 8475 3544 50  0000 C CNN
-F 2 "Button_Switch_THT:SW_Slide_1P2T_CK_OS102011MS2Q" H 8475 3350 50  0001 C CNN
-F 3 "~" H 8475 3350 50  0001 C CNN
-	1    8475 3350
+P 8750 3450
+F 0 "SW1" H 8750 3735 50  0000 C CNN
+F 1 "SW_SPDT" H 8750 3644 50  0000 C CNN
+F 2 "Button_Switch_THT:SW_Slide_1P2T_CK_OS102011MS2Q" H 8750 3450 50  0001 C CNN
+F 3 "~" H 8750 3450 50  0001 C CNN
+	1    8750 3450
 	1    0    0    -1
 $EndComp
@@
 Text GLabel 7550 3250 2    50   Input ~ 0
 TFT_RST
-Text GLabel 7550 4150 2    50   Input ~ 0
-CTP_INT
 $Comp
 L Device:CP_Small C1
@@
 Wire Wire Line
 	7400 3150 8050 3150
-Text Label 7575 3150 0    50   ~ 0
+Text Label 7550 4450 0    50   ~ 0
 SHARP_ILED
 Wire Wire Line
-	8675 3250 8750 3250
+	8950 3350 9025 3350
 Wire Wire Line
-	8750 3250 8750 3050
+	9025 3350 9025 3150
 $Comp
 L Device:R R?
 U 1 1 61C6D8C7
-P 8750 2900
+P 9025 3000
 AR Path="/5E88A377/61C6D8C7" Ref="R?"  Part="1"
 AR Path="/61C6D8C7" Ref="R2"  Part="1"
 AR Path="/5F818C22/61C6D8C7" Ref="R?"  Part="1"
 AR Path="/61C30F00/61C6D8C7" Ref="R?"  Part="1"
-F 0 "R2" V 8675 2925 50  0000 C CNN
-F 1 "10k" V 8750 2900 50  0000 C CNN
-F 2 "Resistor_SMD:R_0402_1005Metric_Pad0.72x0.64mm_HandSolder" V 8680 2900 50  0001 C CNN
-F 3 "~" H 8750 2900 50  0001 C CNN
-	1    8750 2900
+F 0 "R2" V 8950 3025 50  0000 C CNN
+F 1 "10k" V 9025 3000 50  0000 C CNN
+F 2 "Resistor_SMD:R_0402_1005Metric_Pad0.72x0.64mm_HandSolder" V 8955 3000 50  0001 C CNN
+F 3 "~" H 9025 3000 50  0001 C CNN
+	1    9025 3000
 	-1   0    0    -1
 $EndComp
@@
 L power:+3.3V #PWR?
 U 1 1 61C719E6
-P 8750 2500
+P 9025 2600
 AR Path="/5F7FDDC6/61C719E6" Ref="#PWR?"  Part="1"
 AR Path="/61C719E6" Ref="#PWR013"  Part="1"
-F 0 "#PWR013" H 8750 2350 50  0001 C CNN
-F 1 "+3.3V" H 8765 2673 50  0000 C CNN
-F 2 "" H 8750 2500 50  0001 C CNN
-F 3 "" H 8750 2500 50  0001 C CNN
-	1    8750 2500
+F 0 "#PWR013" H 9025 2450 50  0001 C CNN
+F 1 "+3.3V" H 9040 2773 50  0000 C CNN
+F 2 "" H 9025 2600 50  0001 C CNN
+F 3 "" H 9025 2600 50  0001 C CNN
+	1    9025 2600
 	1    0    0    -1
 $EndComp
 Wire Wire Line
-	8750 2750 8750 2500
+	9025 2850 9025 2600
 Wire Wire Line
-	8675 3450 8750 3450
+	8950 3550 9025 3550
 Wire Wire Line
-	8750 3450 8750 3575
+	9025 3550 9025 3675
 $Comp
 L power:GND #PWR?
 U 1 1 61C79EDD
-P 8750 3575
+P 9025 3675
 AR Path="/5F7FDDC6/61C79EDD" Ref="#PWR?"  Part="1"
 AR Path="/61C79EDD" Ref="#PWR014"  Part="1"
-F 0 "#PWR014" H 8750 3325 50  0001 C CNN
-F 1 "GND" H 8755 3402 50  0000 C CNN
-F 2 "" H 8750 3575 50  0001 C CNN
-F 3 "" H 8750 3575 50  0001 C CNN
-	1    8750 3575
+F 0 "#PWR014" H 9025 3425 50  0001 C CNN
+F 1 "GND" H 9030 3502 50  0000 C CNN
+F 2 "" H 9025 3675 50  0001 C CNN
+F 3 "" H 9025 3675 50  0001 C CNN
+	1    9025 3675
 	1    0    0    -1
 $EndComp
@@
 L Device:C C?
 U 1 1 61C7C745
-P 8900 3250
+P 9175 3350
 AR Path="/5F7FDDC6/61C7C745" Ref="C?"  Part="1"
 AR Path="/61C7C745" Ref="C7"  Part="1"
-F 0 "C7" H 9015 3296 50  0000 L CNN
-F 1 "0.1uF" H 9015 3205 50  0000 L CNN
-F 2 "Capacitor_SMD:C_0402_1005Metric_Pad0.74x0.62mm_HandSolder" H 8938 3100 50  0001 C CNN
-F 3 "~" H 8900 3250 50  0001 C CNN
-	1    8900 3250
+F 0 "C7" H 9290 3396 50  0000 L CNN
+F 1 "0.1uF" H 9290 3305 50  0000 L CNN
+F 2 "Capacitor_SMD:C_0402_1005Metric_Pad0.74x0.62mm_HandSolder" H 9213 3200 50  0001 C CNN
+F 3 "~" H 9175 3350 50  0001 C CNN
+	1    9175 3350
 	0    1    1    0
 $EndComp
-Connection ~ 8750 3250
+Connection ~ 9025 3350
 $Comp
 L power:GND #PWR?
 U 1 1 61C7EC98
-P 9200 3250
+P 9475 3350
 AR Path="/5F7FDDC6/61C7EC98" Ref="#PWR?"  Part="1"
 AR Path="/61C7EC98" Ref="#PWR015"  Part="1"
-F 0 "#PWR015" H 9200 3000 50  0001 C CNN
-F 1 "GND" H 9205 3077 50  0000 C CNN
-F 2 "" H 9200 3250 50  0001 C CNN
-F 3 "" H 9200 3250 50  0001 C CNN
-	1    9200 3250
+F 0 "#PWR015" H 9475 3100 50  0001 C CNN
+F 1 "GND" H 9480 3177 50  0000 C CNN
+F 2 "" H 9475 3350 50  0001 C CNN
+F 3 "" H 9475 3350 50  0001 C CNN
+	1    9475 3350
 	0    -1   -1   0
 $EndComp
 Wire Wire Line
-	9200 3250 9050 3250
+	9475 3350 9325 3350
 Wire Wire Line
 	9500 1650 10150 1650
-Text Label 7550 3550 0    50   ~ 0
+Text Label 7550 4150 0    50   ~ 0
 GPIO17
-Text Label 7550 4450 0    50   ~ 0
-GPIO32
+Text Label 7675 3150 0    50   ~ 0
+GPIO16
 Text Label 7550 4550 0    50   ~ 0
 GPIO33
-$Comp
-L Connector:Conn_01x04_Male J3
-U 1 1 61C918EE
-P 3625 4050
-F 0 "J3" H 3597 3932 50  0000 R CNN
-F 1 "GPIO expanded" H 3597 4023 50  0000 R CNN
-F 2 "SnapEDA Library:JST_SM04B-SRSS-TB(LF)(SN)" H 3625 4050 50  0001 C CNN
-F 3 "~" H 3625 4050 50  0001 C CNN
-	1    3625 4050
-	-1   0    0    -1
-$EndComp
 Wire Wire Line
 	3425 4250 3000 4250
@@
 Wire Wire Line
 	3425 3950 3000 3950
-Text Label 3275 4050 2    50   ~ 0
-GPIO16
 Text Label 3275 3950 2    50   ~ 0
+GPIO16
+Text Label 3275 4050 2    50   ~ 0
 GPIO15
-Text Label 3275 4250 2    50   ~ 0
-GPIO32
 Text Label 3275 4150 2    50   ~ 0
+GPIO17
+Text Label 3275 4250 2    50   ~ 0
 GPIO33
 $Comp
@@
 $EndBitmap
 Wire Wire Line
-	8275 3450 8275 3350
-Wire Wire Line
-	7400 3450 8275 3450
-Wire Wire Line
 	7400 3350 7875 3350
 Text Label 7875 3350 0    50   ~ 0
@@
 Text Label 4650 6575 3    50   ~ 0
 IO0
+Text GLabel 8050 4050 2    50   Input ~ 0
+MODBUS_TXD
+Text GLabel 8050 4350 2    50   Input ~ 0
+MODBUS_EN
+Text GLabel 8050 4250 2    50   Input ~ 0
+MODBUS_RXD
+Text GLabel 7550 3550 2    50   Input ~ 0
+CTP_INT
+Wire Wire Line
+	7550 4150 7400 4150
+Wire Wire Line
+	7400 4350 8050 4350
+Wire Wire Line
+	7400 3450 8550 3450
+$Comp
+L Connector:Conn_01x04_Male J3
+U 1 1 61C918EE
+P 3625 4150
+F 0 "J3" H 3597 4032 50  0000 R CNN
+F 1 "GPIO expanded" H 3597 4123 50  0000 R CNN
+F 2 "SnapEDA Library:JST_SM04B-SRSS-TB(LF)(SN)" H 3625 4150 50  0001 C CNN
+F 3 "~" H 3625 4150 50  0001 C CNN
+	1    3625 4150
+	-1   0    0    1
+$EndComp
+Wire Wire Line
+	9500 1350 10150 1350
+$Comp
+L power:+5V #PWR?
+U 1 1 5F99E8D0
+P 10075 3750
+AR Path="/5E88A377/5F99E8D0" Ref="#PWR?"  Part="1"
+AR Path="/5F99E8D0" Ref="#PWR020"  Part="1"
+AR Path="/5F818C22/5F99E8D0" Ref="#PWR?"  Part="1"
+F 0 "#PWR020" H 10075 3600 50  0001 C CNN
+F 1 "+5V" H 10090 3923 50  0000 C CNN
+F 2 "" H 10075 3750 50  0001 C CNN
+F 3 "" H 10075 3750 50  0001 C CNN
+	1    10075 3750
+	-1   0    0    -1
+$EndComp
 $EndSCHEMATC
