File: Max485 wth translator.sch (KiCad schematic (older format))
At the start: 10 parts, among them J6 MODBUS RTU, U3 MAX3485

Commit message: PCB completed
Connections:
- wire segments 44 -> 43
Changed lines of the file:
@@
 L power:GND #PWR?
 U 1 1 61C53454
-P 6475 3175
+P 6475 4550
 AR Path="/5E88A377/61C53454" Ref="#PWR?"  Part="1"
 AR Path="/61C53454" Ref="#PWR?"  Part="1"
 AR Path="/5F818C22/61C53454" Ref="#PWR?"  Part="1"
 AR Path="/61C30F00/61C53454" Ref="#PWR028"  Part="1"
-F 0 "#PWR028" H 6475 2925 50  0001 C CNN
-F 1 "GND" H 6480 3002 50  0000 C CNN
-F 2 "" H 6475 3175 50  0001 C CNN
-F 3 "" H 6475 3175 50  0001 C CNN
-	1    6475 3175
-	-1   0    0    1
+F 0 "#PWR028" H 6475 4300 50  0001 C CNN
+F 1 "GND" H 6480 4377 50  0000 C CNN
+F 2 "" H 6475 4550 50  0001 C CNN
+F 3 "" H 6475 4550 50  0001 C CNN
+	1    6475 4550
+	1    0    0    -1
 $EndComp
 Wire Wire Line
@@
 P 7525 3975
 F 0 "J6" H 7443 4292 50  0000 C CNN
-F 1 "MODBUS RTU" H 7443 4201 50  0000 C CNN
+F 1 "MODBUS RTU" H 7550 4200 50  0000 C CNN
 F 2 "SnapEDA Library:JST_SM03B-SRSS-TB(LF)(SN)" H 7525 3975 50  0001 C CNN
 F 3 "~" H 7525 3975 50  0001 C CNN
 	1    7525 3975
-	1    0    0    1
+	1    0    0    -1
 $EndComp
 Wire Wire Line
 	7325 4075 6475 4075
 Wire Wire Line
-	7325 3975 7125 3975
-Wire Wire Line
-	7125 3975 7125 3625
-Wire Wire Line
-	7125 3625 6475 3625
-Wire Wire Line
 	7325 3875 7250 3875
-Wire Wire Line
-	7250 3875 7250 3775
 $Comp
 L power:GND #PWR?
 U 1 1 61C5346A
-P 7250 3775
+P 7125 3975
 AR Path="/5E88A377/61C5346A" Ref="#PWR?"  Part="1"
 AR Path="/61C5346A" Ref="#PWR?"  Part="1"
 AR Path="/5F818C22/61C5346A" Ref="#PWR?"  Part="1"
 AR Path="/61C30F00/61C5346A" Ref="#PWR030"  Part="1"
-F 0 "#PWR030" H 7250 3525 50  0001 C CNN
-F 1 "GND" H 7255 3602 50  0000 C CNN
-F 2 "" H 7250 3775 50  0001 C CNN
-F 3 "" H 7250 3775 50  0001 C CNN
-	1    7250 3775
-	-1   0    0    1
+F 0 "#PWR030" H 7125 3725 50  0001 C CNN
+F 1 "GND" H 7130 3802 50  0000 C CNN
+F 2 "" H 7125 3975 50  0001 C CNN
+F 3 "" H 7125 3975 50  0001 C CNN
+	1    7125 3975
+	0    1    1    0
 $EndComp
 Text Label 5225 4075 2    50   ~ 0
@@
 Text Label 5175 3625 2    50   ~ 0
 A
-Text Label 3225 4075 2    50   ~ 0
-MODBUS_RXD
-Text Label 3225 3975 2    50   ~ 0
-MODBUS_EN
-Text Label 3225 3775 2    50   ~ 0
-MODBUS_TXD
 Wire Wire Line
 	2825 3775 3500 3775
@@
 L power:+3.3V #PWR029
 U 1 1 61C6EF46
-P 6475 4550
-F 0 "#PWR029" H 6475 4400 50  0001 C CNN
-F 1 "+3.3V" H 6490 4723 50  0000 C CNN
-F 2 "" H 6475 4550 50  0001 C CNN
-F 3 "" H 6475 4550 50  0001 C CNN
-	1    6475 4550
-	-1   0    0    1
-$EndComp
+P 6475 3175
+F 0 "#PWR029" H 6475 3025 50  0001 C CNN
+F 1 "+3.3V" H 6490 3348 50  0000 C CNN
+F 2 "" H 6475 3175 50  0001 C CNN
+F 3 "" H 6475 3175 50  0001 C CNN
+	1    6475 3175
+	1    0    0    -1
+$EndComp
+Text GLabel 2825 3775 0    50   Input ~ 0
+MODBUS_TXD
+Text GLabel 2825 3975 0    50   Input ~ 0
+MODBUS_EN
+Text GLabel 2825 4075 0    50   Input ~ 0
+MODBUS_RXD
+Wire Wire Line
+	6475 3625 7250 3625
+Wire Wire Line
+	7250 3625 7250 3875
+Wire Wire Line
+	7325 3975 7125 3975
 $EndSCHEMATC

Commit message: Schematics change
Parts:
- J6: MPN (none) -> JST_SM03B-SRSS-TB(LF)(SN)
- U3: MPN (none) -> MAX3485
Changed lines of the file:
@@
 F 2 "SnapEDA Library:JST_SM03B-SRSS-TB(LF)(SN)" H 7525 3975 50  0001 C CNN
 F 3 "~" H 7525 3975 50  0001 C CNN
+F 4 "JST_SM03B-SRSS-TB(LF)(SN)" H 7525 3975 50  0001 C CNN "MPN"
 	1    7525 3975
 	1    0    0    -1
@@
 F 2 "Package_SO:SOIC-8_3.9x4.9mm_P1.27mm" H 4600 3275 50  0001 C CNN
 F 3 "https://datasheets.maximintegrated.com/en/ds/MAX3483-MAX3491.pdf" H 4600 4025 50  0001 C CNN
+F 4 "MAX3485" H 4600 3975 50  0001 C CNN "MPN"
 	1    4600 3975
 	1    0    0    1
