File: _autosave-ESP32_BoardV1.sch (KiCad schematic (older format))
At the start: 30 parts, among them J1 Barrel_Jack_Switch, J2 ISP, J3 GPIO expanded, J4 sensor, J5 I2C extended, J7 Display, Q1 UMH3N, SW1 SW_SPDT, U1 AZ1117-3.3, U2 ESP32-WROOM-32E(8MB)

Commit message: Final draft with GERBER and Manufacturing Data
Parts:
- added U?: ESP32-WROOM-32D, RF_Module:ESP32-WROOM-32, symbol RF_Module:ESP32-WROOM-32D
