File: ESP32_BoardV1.kicad_pcb (KiCad board)
At the start: 2 copper layers, 120 x 60 mm, 43 parts, among them J1 Barrel_Jack_Switch, J2 ISP, J3 GPIO expanded, J4 sensor, J5 I2C extended, J6 MODBUS RTU, J7 Display, Q1 UMH3N, Q2 SS8050-G, SW1 SW_SPDT, U1 AZ1117-3.3, U2 ESP32-WROOM-32E(8MB), U3 MAX3485

Commit message: Final draft with GERBER and Manufacturing Data
Parts:
- removed Q2: SS8050-G, Package_TO_SOT_SMD:SOT-23
- removed R12: 10K, Resistor_SMD:R_0402_1005Metric_Pad0.72x0.64mm_HandSolder
- removed R13: 10R, Resistor_SMD:R_0402_1005Metric_Pad0.72x0.64mm_HandSolder
- added C11: 4.7uF, Capacitor_SMD:C_0402_1005Metric, F.Cu at (170.6, 143.4)
- added C13: 1uF, Capacitor_SMD:C_0402_1005Metric, F.Cu at (173.1, 136.1)
- added D3: D_Schottky, Diode_SMD:D_SOD-123F, F.Cu at (175.9, 141.2)
- added L1: 4.7uF, Inductor_SMD:L_1008_2520Metric, F.Cu at (173.3, 141.1)
- added U4: TPS61169DCKR, Package_TO_SOT_SMD:SOT-353_SC-70-5, F.Cu at (170.5, 141.2)
- C2: footprint Capacitor_Tantalum_SMD:CP_EIA-3528-21_Kemet-B -> Capacitor_SMD:CP_Elec_6.3x5.4
- Q1: value UMH3N -> Taiyo Yuden
- R1, R3, R4, R5: value 10K -> 10k
- R11: value 10K -> 5R
- moved C7 37.5 mm to (149.3, 103.4)
- moved R2 37.5 mm to (149.3, 102.4)
- moved SW1 37.5 mm to (147.0, 97.7)
- moved Q1 29.3 mm to (102.9, 103.5), turned to 90 degrees
- moved J2 28.7 mm to (95.2, 97.2), turned to 90 degrees
- moved R11 16.5 mm to (171.3, 134.3), turned to 0 degrees
- moved C2 8.82 mm to (158.2, 137.2), turned to 90 degrees
- moved C1 2.93 mm to (167.2, 147.6), turned to -90 degrees
- moved C10 2.80 mm to (171.3, 131.8)
- moved C9 2.80 mm to (171.3, 132.8)
Connections:
- J2 pad 1: /UART0_RXD -> /UART0_TXD
- J2 pad 2: /UART0_TXD -> /UART0_RXD
- J2 pad 3: /DTR -> /RESET
- J2 pad 5: /RESET -> /DTR
- J7 pad 1: +3V3 -> /LED_A
- R11 pad 1: Net-(Q2-Pad1) -> GND
- R11 pad 2: /BL_CONTRL -> /LED_K
Routing:
- net Net-(SW1-Pad2): track 19.3 -> 53.6 mm
- net /RESET: track 40.9 -> 59.2 mm
- net Net-(Q2-Pad3): track 17.8 -> 0.00 mm
- net /BL_CONTRL: track 50.3 -> 64.9 mm
- net /LED_A: track 0.00 -> 13.6 mm
- net MODBUS_TXD: track 57.2 -> 44.5 mm, vias 2 -> 0
- net CTP_SDA: track 142.5 -> 134.1 mm, vias 4 -> 3
- net CTP_SCL: track 144.6 -> 136.7 mm, vias 4 -> 3
- net +3V3: track 37.0 -> 44.7 mm, vias 3 -> 2
- net /LED_K: track 2.16 -> 8.56 mm
- net GND: track 82.6 -> 76.2 mm, vias 56 -> 59
- net CTP_INT: track 86.3 -> 92.3 mm
- net Net-(D3-Pad2): track 0.00 -> 5.14 mm
- net TFT_CS: track 91.4 -> 95.7 mm
- net MODBUS_EN: track 54.2 -> 50.7 mm, vias 0 -> 2
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
Commit message: Change 1/1/21
Parts:
- added C12: 1nF, Capacitor_SMD:C_0402_1005Metric, F.Cu at (168.5, 121.7)
- added R12: 10k, Resistor_SMD:R_0402_1005Metric_Pad0.72x0.64mm_HandSolder, F.Cu at (171.1, 116.7)
- C4, C5, C6, C8: footprint Capacitor_SMD:C_0805_2012Metric -> Capacitor_SMD:C_0402_1005Metric_Pad0.74x0.62mm_HandSolder
- H1, H2, H3, H4: footprint MountingHole:MountingHole_3.5mm_Pad_Via -> MountingHole:MountingHole_4.3mm_M4_Pad_Via
- L1: value 4.7uF -> 4.7uH
- Q1: value Taiyo Yuden -> UMH3N
- R1, R3, R4, R5: value 10k -> 10K; footprint Resistor_SMD:R_0805_2012Metric -> Resistor_SMD:R_0402_1005Metric_Pad0.72x0.64mm_HandSolder
- R6: footprint Resistor_SMD:R_1206_3216Metric -> Resistor_SMD:R_0402_1005Metric_Pad0.72x0.64mm_HandSolder
- R7, R8: value 5k -> 10k; footprint Resistor_SMD:R_0805_2012Metric -> Resistor_SMD:R_0402_1005Metric_Pad0.72x0.64mm_HandSolder
- moved C5 2.70 mm to (93.0, 140.3)
- moved R9 2.60 mm to (166.9, 113.7)
- moved R10 2.60 mm to (166.9, 116.2)
- moved R1 1.80 mm to (93.0, 139.2)
- moved R7 1.80 mm to (133.3, 142.5)
- moved R8 1.80 mm to (138.0, 142.5)
- moved C8 1.49 mm to (139.0, 125.1)
- moved C4 0.90 mm to (93.0, 138.1)
- moved U1 0.55 mm to (173.5, 149.8)
- moved U4 0.10 mm to (170.4, 141.2)
Connections:
- J2 pad 1: /UART0_TXD -> /UART0_RXD
- J2 pad 2: /UART0_RXD -> /UART0_TXD
- J7 pad 37: +3V3 -> Net-(J7-Pad37)
Routing:
- net +3V3: track 44.7 -> 35.8 mm
- net /RESET: track 59.2 -> 55.8 mm
- net Net-(J7-Pad37): track 0.00 -> 1.97 mm
- net GND: track 76.2 -> 77.5 mm, vias 59 -> 58
- net /Modubus/A: track 26.3 -> 25.4 mm
- net CTP_SDA: track 134.1 -> 133.4 mm
