File: Max485 wth translator.kicad_sch (KiCad schematic)
At the start: 10 parts, among them J6 MODBUS RTU, U3 MAX3485

Commit message: Final draft with GERBER and Manufacturing Data
Parts:
- C8: footprint Capacitor_SMD:C_0402_1005Metric -> Capacitor_SMD:C_0402_1005Metric_Pad0.74x0.62mm_HandSolder; MPN 04026D104KAT2A -> (none); Manufacturer KYOCERA AVX -> (none)
- D2: symbol Device:D_TVS_x2_AAC -> Device:D_TVS_Dual_AAC; MPN SM712 -> (none); Manufacturer MDD -> (none)
- J6: MPN SM03B-SRSS-TB(LF)(SN) -> JST_SM03B-SRSS-TB(LF)(SN); Manufacturer JST Sales America Inc. -> (none)
- R3, R4, R5: value 10k -> 10K; MPN RMCF0402FT5K10 -> (none); Manufacturer Stackpole Electronics Inc -> (none)
- R6: MPN SS8050-G -> (none); Manufacturer TE Connectivity Passive Product -> (none)
- R7, R8: value 5k -> 10k; MPN CRGCQ0402F120R -> (none); Manufacturer Stackpole Electronics Inc -> (none)
- U3: MPN ESP32-WROOM-32E(8MB) -> MAX3485; Manufacturer Analog Devices Inc./Maxim Integrated -> (none)

Commit message: Change 1/1/21
Parts:
- R7, R8: value 10k -> 5K
Changed lines of the file:
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@@
     (in_bom yes) (on_board yes)
     (property "Reference" "R8" (id 0) (at 166.37 108.585 90))
-    (property "Value" "10k" (id 1) (at 164.465 109.22 90))
+    (property "Value" "5K" (id 1) (at 164.465 109.22 90))
     (property "Footprint" "Resistor_SMD:R_0402_1005Metric_Pad0.72x0.64mm_HandSolder" (id 2) (at 166.243 109.22 90)
       (effects (font (size 1.27 1.27)) hide)
@@
     (in_bom yes) (on_board yes)
     (property "Reference" "R7" (id 0) (at 166.37 85.725 90))
-    (property "Value" "10k" (id 1) (at 164.465 86.36 90))
+    (property "Value" "5K" (id 1) (at 164.465 86.36 90))
     (property "Footprint" "Resistor_SMD:R_0402_1005Metric_Pad0.72x0.64mm_HandSolder" (id 2) (at 166.243 86.36 90)
       (effects (font (size 1.27 1.27)) hide)
