File: ESP32_BoardV1.kicad_sch (KiCad schematic)
At the start: 33 parts, among them J1 Barrel_Jack_Switch, J2 ISP, J3 GPIO expanded, J4 sensor, J5 I2C extended, J7 Display, Q1 UMH3N, Q2 SS8050-G, SW1 SW_SPDT, U1 AZ1117-3.3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

Commit message: Final draft with GERBER and Manufacturing Data
Parts:
- removed Q2: SS8050-G, Package_TO_SOT_SMD:SOT-23, symbol Device:Q_NPN_BEC
- removed R12: 10k, Resistor_SMD:R_0402_1005Metric_Pad0.72x0.64mm_HandSolder, symbol Device:R
- removed R13: 10R, Resistor_SMD:R_0402_1005Metric_Pad0.72x0.64mm_HandSolder, symbol Device:R
- added C11: 4.7uF, Capacitor_SMD:C_0402_1005Metric, symbol Device:C
- added C13: 1uF, Capacitor_SMD:C_0402_1005Metric, symbol Device:C
- added D3: D_Schottky, Diode_SMD:D_SOD-123F, symbol Device:D_Schottky
- added JP1: SolderJumper_2_Open, Resistor_SMD:R_0402_1005Metric_Pad0.72x0.64mm_HandSolder, symbol Jumper:SolderJumper_2_Open
- added L1: 4.7uH, Inductor_SMD:L_1008_2520Metric, symbol Device:L_Small
- added U4: TPS61169DCKR, Package_TO_SOT_SMD:SOT-353_SC-70-5, symbol TPS61169DCKR:TPS61169DCKR
- C1: symbol Device:CP_Small -> Device:C_Polarized_Small; MPN AVE106M16A12T-F -> (none); Manufacturer Cornell Dubilier Electronics (CDE) -> (none)
- C10, C5, C6, C7: footprint Capacitor_SMD:C_0402_1005Metric -> Capacitor_SMD:C_0402_1005Metric_Pad0.74x0.62mm_HandSolder; MPN 04026D104KAT2A -> (none); Manufacturer KYOCERA AVX -> (none)
- C2: footprint Capacitor_Tantalum_SMD:CP_EIA-3528-21_Kemet-B -> Capacitor_SMD:CP_Elec_6.3x5.4; symbol Device:CP -> Device:C_Polarized_Small; MPN T491B107M010AT -> (none); Manufacturer KEMET -> (none)
- C3: symbol Device:CP_Small -> Device:C_Polarized_Small; MPN UWT1A220MCL1GB -> (none); Manufacturer Nichicon -> (none)
- C4, C9: footprint Capacitor_SMD:C_0402_1005Metric -> Capacitor_SMD:C_0402_1005Metric_Pad0.74x0.62mm_HandSolder; MPN GRM155R60J106ME15D -> (none); Manufacturer Murata Electronics -> (none)
- D1: MPN SMBJ5.0CA-13-F -> (none); Manufacturer Diodes Incorporated -> (none)
- F1: MPN C1Q 2 -> (none); Manufacturer Bel Fuse Inc. -> (none)
- H1, H2, H3, H4: MPN n/C -> (none); Manufacturer N/C -> (none)
- J1: MPN PJ-030DH-SMT-TR -> (none); Manufacturer CUI Devices -> (none)
- J2: MPN PR20206VBNN -> (none); Manufacturer METZ CONNECT USA Inc. -> (none)
- J3, J5: MPN SM04B-SRSS-TB(LF)(SN) -> JST_SM04B-SRSS-TB(LF)(SN); Manufacturer JST Sales America Inc. -> (none)
- J4: MPN SM05B-SRSS-TB(LF)(SN) -> JST_SM05B-SRSS-TB(LF)(SN); Manufacturer JST Sales America Inc. -> (none)
- J7: MPN FH12-40S-0.5SVA(55) -> (none); Manufacturer Hirose Electric Co Ltd -> (none)
- Q1: MPN FH12-40S-0.5SVA(55) -> (none); Manufacturer NXP USA Inc. -> (none)
- R1: value 10k -> 10K; MPN RMCF0402FT5K10 -> (none); Manufacturer Stackpole Electronics Inc -> (none)
- R10, R2, R9: MPN RMCF0402FT5K10 -> (none); Manufacturer Stackpole Electronics Inc -> (none)
- R11: value 10k -> 5R; MPN RMCF0402FT5K10 -> (none); Manufacturer Stackpole Electronics Inc -> (none)
- SW1: MPN RMCF0402FT10R0 -> (none); Manufacturer TE Connectivity ALCOSWITCH Switches -> (none)
- U1: MPN 1825232-1 -> AZ1117-3.3; Manufacturer Diodes Incorporated -> (none)
- U2: symbol ESP32_BoardV1-rescue:ESP32-WROOM-32D-RF_Module -> RF_Module:ESP32-WROOM-32D; MPN AZ1117IH-3.3TRG1 -> ESP32-WROOM-32; Manufacturer Espressif Systems -> (none)
Connections:
- net +3V3: now also JP1.1 (A); no longer J3.4 (Pin_4), J5.1 (Pin_1), J7.1 (Pin_1)
- net +5V: now also C11.1, L1.1, U4.5 (VIN)
- net BL_CONTRL: now also U4.4 (CTRL); no longer R11.2, U2.16 (IO13)
- net GND: now also R11.1, C11.2, C13.2, U4.2 (GND)
- net LED_K: now also R11.2, U4.3 (FB); no longer J7.2 (Pin_2)
- new net: D3.2 (A), L1.2, U4.1 (SW)
- new net GPIO16: J3.4 (Pin_4), U2.16 (IO13)
- new net LED_A: C13.1, D3.1 (K)
- new net VCC: J5.1 (Pin_1), JP1.2 (B)
- no-connect marks 12 -> 8
Other:
- moved on the sheet: C4, C6, J2, J3, Q1A, Q1B

Commit message: Change 1/1/21
Parts:
- removed JP1: SolderJumper_2_Open, Resistor_SMD:R_0402_1005Metric_Pad0.72x0.64mm_HandSolder, symbol Jumper:SolderJumper_2_Open
- added C12: 1nF, Capacitor_SMD:C_0402_1005Metric, symbol Device:C
- added R12: 10k, Resistor_SMD:R_0402_1005Metric_Pad0.72x0.64mm_HandSolder, symbol Device:R
Connections:
- net VCC is gone; now on net +3V3: J5.1 (Pin_1)
- net +3V3: now also J3.4 (Pin_4), C12.1, R12.1; no longer J7.37 (Pin_37)
- net BL_CONTRL: now also U2.16 (IO13)
- net DTR: now also J2.5 (Pin_5); no longer J2.3 (Pin_3)
- net GND: now also C12.2
- net LED_A: now also J7.1 (Pin_1)
- net LED_K: now also J7.2 (Pin_2)
- net RESET: now also J2.3 (Pin_3); no longer J2.5 (Pin_5)
- removed net GPIO16: J3.4 (Pin_4), U2.16 (IO13)
- new net: J7.37 (Pin_37), R12.2

Commit message: added gebr and DFM data
Other:
- company: SMB ElectroTech -> (none)
